File: pcb/pcb.kicad_pcb (KiCad board)
At the start: 2 copper layers, 208.2 x 21 mm, 89 parts, among them J1 ER-TFT0.96-1, J2 USB_C_Receptacle, J3 Conn_01x04, J4 Conn_01x03, J5 Conn_01x35, SW1 SKQG, SW2 SKQG, SW3 SKQG, SW4 SKQG, SW5 SKQG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

Commit message: pcb: rev 0.2
Parts:
- removed L1: 300R, Inductor_SMD:L_0603_1608Metric
- added C35: 100nF, Capacitor_SMD:C_0402_1005Metric, F.Cu at (166.4, 90.7)
- added C36: 100nF, Capacitor_SMD:C_0402_1005Metric, F.Cu at (166.4, 91.7)
- added C37: 100nF, Capacitor_SMD:C_0402_1005Metric, F.Cu at (166.4, 92.7)
- added C38: 100nF, Capacitor_SMD:C_0402_1005Metric, F.Cu at (166.4, 93.7)
- added C39: 100nF, Capacitor_SMD:C_0402_1005Metric, F.Cu at (166.4, 96.7)
- added C40: 100nF, Capacitor_SMD:C_0402_1005Metric, F.Cu at (166.4, 97.7)
- added C41: 100nF, Capacitor_SMD:C_0402_1005Metric, F.Cu at (162.4, 90.1)
- added TP3: TestPoint, TestPoint:TestPoint_Pad_D1.0mm, F.Cu at (179.1, 82.1)
- added U9: CBTL02043A, Package_DFN_QFN:WQFN-20-1EP_2.5x4.5mm_P0.5mm_EP1x2.9mm, F.Cu at (162.4, 94.3)
- C16, C17: value 220nF -> 100nF
- J5: value Conn_01x35 -> Conn_01x40_MountingPin; footprint Connector_PinHeader_1.27mm:PinHeader_1x35_P1.27mm_Vertical -> footprints:Hirose_FH12-40S-0.5SH_1x40-1MP_P0.50mm_Horizontal_Reversed; moved to B.Cu
- L4: footprint Inductor_SMD:L_Vishay_IHLP-1212 -> Inductor_SMD:L_Vishay_IHLP-1616
- R16: value 200K -> 36K
- R17: value 100K -> 8.25K
- R20: value 100K -> 10K
- moved J4 77.6 mm to (213.4, 81.8)
- moved C2 75.4 mm to (228.1, 83.4)
- moved U2 75.4 mm to (228.1, 96.9)
- moved C10 75.4 mm to (223.2, 95.5)
- moved C11 75.4 mm to (229.1, 89.2)
- moved C12 75.4 mm to (228.5, 93.4)
- moved C14 75.4 mm to (224.8, 97.7)
- moved C3 75.4 mm to (222.8, 84.0)
- moved C6 75.4 mm to (221.4, 95.5)
- moved C7 75.4 mm to (221.8, 84.0)
- moved C8 75.4 mm to (218.8, 93.3)
- moved C9 75.4 mm to (220.1, 95.5)
- moved R1 75.4 mm to (224.3, 85.5)
- moved R4 75.4 mm to (222.9, 97.8)
- moved R5 75.4 mm to (221.9, 97.8)
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Connections:
- net /TYPEC_RX2N renamed /TX2N
- net /TYPEC_RX2P renamed /TX2P
- C16 pad 2: /DP0N -> Net-(C16-Pad2)
- C17 pad 2: /DP0P -> Net-(C17-Pad2)
- J2 pad A2: unconnected-(J2-PadA2) -> /RX1P
- J2 pad A3: unconnected-(J2-PadA3) -> /RX1N
- J2 pad A4: Net-(J2-PadA4) -> VBUS
- J2 pad A6: unconnected-(J2-PadA6) -> USB_DP
- J2 pad A7: unconnected-(J2-PadA7) -> USB_DN
- J2 pad A9: Net-(J2-PadA4) -> VBUS
- J2 pad B10: unconnected-(J2-PadB10) -> /TX1N
- J2 pad B11: unconnected-(J2-PadB11) -> /TX1P
- J2 pad B2: /DP1P -> /RX2P
- J2 pad B3: /DP1N -> /RX2N
- J2 pad B4: Net-(J2-PadA4) -> VBUS
- J2 pad B7: USB_DM -> USB_DN
- J2 pad B9: Net-(J2-PadA4) -> VBUS
- J5 pad 26: /BL_ON -> unconnected-(J5-Pad26)
- J5 pad 31: unconnected-(J5-Pad31) -> GND
- J5 pad 32: +12V -> GND
- J5 pad 33: +12V -> unconnected-(J5-Pad33)
- J5 pad 35: unconnected-(J5-Pad35) -> +12V
- J5 pad 6: Net-(C32-Pad2) -> +3V3
- R5 pad 1: USB_DM -> USB_DN
- U1 pad 17: /GPIO14 -> TYPEC_ORI
- U3 pad 3: USB_DM -> USB_DN
- U3 pad 4: USB_DM -> USB_DN
- U3 pad 5: Net-(J2-PadA4) -> VBUS
- U5 pad A2: Net-(J2-PadA4) -> unconnected-(U5-PadA2)
Routing:
- net KEY5: track 13.4 -> 103.9 mm, vias 0 -> 2
- net KEY4: track 30.0 -> 119.5 mm, vias 0 -> 2
- net KEY3: track 46.2 -> 134.6 mm, vias 0 -> 2
- net KEY2: track 64.6 -> 152.9 mm, vias 0 -> 2
- net LED3: track 44.3 -> 132.4 mm, vias 0 -> 2
- net LED1: track 59.5 -> 147.4 mm, vias 0 -> 2
- net KEY1: track 93.3 -> 180.7 mm, vias 0 -> 2
- net LED4: track 40.4 -> 127.0 mm, vias 0 -> 2
- net LED2: track 56.2 -> 141.9 mm, vias 0 -> 2
- net TYPEC_ORI: track 0.00 -> 73.1 mm, vias 0 -> 4
- net +3V3: track 198.6 -> 259.6 mm, vias 17 -> 21
- net USB_DN: track 0.00 -> 54.4 mm, vias 0 -> 1
- net GND: track 88.5 -> 140.3 mm, vias 118 -> 111
- net USB_DM: track 47.7 -> 0.00 mm, vias 1 -> 0
- net Net-(J2-PadA4): track 41.6 -> 0.00 mm, vias 2 -> 0
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- added copper zone on In1.Cu, net GND
- added copper zone on In2.Cu, net GND
Other:
- board size 208.2 x 21 mm -> 207.4 x 21 mm
- copper layers 2 -> 4
- board text added: "Board Thickness: 1.0 mm Board Layer Count: 4 85 ohm Diff-Pair (DP): 0.1mm sep, 0.2mm width 90 ohm Diff-Pair (USB): 0.1mm sep, 0.18mm width 100 ohm Diff-Pair (LVDS): 0.1mm sep, 0.14mm width"
- board text added: "GND RX TX 3V3"
- board text added: "R0.2 (C) Wenting 2021"
- board text removed: "12V"
- board text removed: "3V TX RX GND"
- board text removed: "3V3"
- board text removed: "BLON"
- board text removed: "Board Thickness: 0.8 mm Board Layer Count: 2 85 ohm Diff-Pair (DP): 0.127mm sep, 0.8mm width 90 ohm Diff-Pair (USB): 0.127mm sep, 0.65mm width 100 ohm Diff-Pair (LVDS): 0.127mm sep, 0.45mm width"
- board text removed: "CLK+"
- board text removed: "CLK-"
- board text removed: "D0+"
- board text removed: "D0-"
- board text removed: "D1+"
- board text removed: "D1-"
- board text removed: "D2+"
- board text removed: "D2-"
- board text removed: "GND"
- board text removed: "PWM"
- board text removed: "R0.1 (C) Wenting 2021"
- board text removed: "SCL"
- board text removed: "SDA"
