File: pcb/pcb.kicad_sch (KiCad schematic)
At the start: 89 parts, among them J1 ER-TFT0.96-1, J2 USB_C_Receptacle, J3 Conn_01x04, J4 Conn_01x03, J5 Conn_01x35, SW1 SKQG, SW2 SKQG, SW3 SKQG, SW4 SKQG, SW5 SKQG, U1 RP2040, U2 FM25Q04-DN-T-G, U3 USBLC6-2P6, U4 SY8008, U5 FUSB302UCX, U6 PTN3460, U7 SY7152, U8 NX3P1108UK, Y1 24MHz

Commit message: pcb: rev 0.2
Parts:
- removed J5: Conn_01x35, Connector_PinHeader_1.27mm:PinHeader_1x35_P1.27mm_Vertical, symbol Connector_Generic:Conn_01x35
- removed L1: 300R, Inductor_SMD:L_0603_1608Metric, symbol Device:L
- added C35, C36, C37, C38, C39, C40, C41: 100nF, Capacitor_SMD:C_0402_1005Metric, symbol Device:C
- added J5: Conn_01x40_MountingPin, footprints:Hirose_FH12-40S-0.5SH_1x40-1MP_P0.50mm_Horizontal_Reversed, symbol Connector_Generic_MountingPin:Conn_01x40_MountingPin
- added TP3: TestPoint, TestPoint:TestPoint_Pad_D1.0mm, symbol Connector:TestPoint
- added U9: CBTL02043A, Package_DFN_QFN:WQFN-20-1EP_2.5x4.5mm_P0.5mm_EP1x2.9mm, symbol Analog_Switch:CBTL02043A
- C16, C17: value 220nF -> 100nF
- L4: footprint Inductor_SMD:L_Vishay_IHLP-1212 -> Inductor_SMD:L_Vishay_IHLP-1616
- R16: value 200K -> 36K
- R17: value 100K -> 8.25K
- R20: value 100K -> 10K
Connections:
- net USB_DM is gone; now on net USB_DN: J2.B7 (D-), R5.1, U3.3 (I/O2), U3.4 (I/O2)
- net +12V: now also J5.34 (Pin_34), J5.35 (Pin_35), J5.36 (Pin_36), J5.37 (Pin_37), J5.38 (Pin_38)
- net +3V3: now also C41.1, J5.6 (Pin_6), U9.1 (VDD), U9.10 (VDD), U9.6 (VDD)
- net BL_ON: now also TP3.1
- net DDC_CLK: now also J5.8 (Pin_8)
- net DDC_DATA: now also J5.9 (Pin_9)
- net DP0N: now also U9.7 (A1_P); no longer C16.2
- net DP0P: now also U9.8 (A1_N); no longer C17.2
- net DP1N: now also U9.3 (A0_P); no longer J2.B3 (TX2-)
- net DP1P: now also U9.4 (A0_N); no longer J2.B2 (TX2+)
- net GND: now also C41.2, J5.1 (Pin_1), J5.10 (Pin_10), J5.11 (Pin_11), J5.15 (Pin_15), J5.18 (Pin_18), J5.21 (Pin_21), J5.24 (Pin_24), J5.28 (Pin_28), J5.29 (Pin_29), J5.30 (Pin_30), J5.31 (Pin_31), J5.32 (Pin_32), J5.40 (Pin_40), J5.MP (MountPin), U9.11 (GND), U9.20 (GND), U9.21 (GND), U9.5 (GND), U9.9 (SEL)
- net RCLKIN+: now also J5.23 (Pin_23)
- net RCLKIN-: now also J5.22 (Pin_22)
- net RIN0+: now also J5.14 (Pin_14)
- net RIN0-: now also J5.13 (Pin_13)
- net RIN1+: now also J5.17 (Pin_17)
- net RIN1-: now also J5.16 (Pin_16)
- net RIN2+: now also J5.20 (Pin_20)
- net RIN2-: now also J5.19 (Pin_19)
- net USB_DP: now also J2.A6 (D+)
- net VBUS: now also J2.A4 (VBUS), J2.A9 (VBUS), J2.B4 (VBUS), J2.B9 (VBUS), U3.5 (VBUS)
- net VDIM: now also J5.25 (Pin_25)
- net at C32.2, U8.A1 (VOUT): now also J5.3 (Pin_3), J5.4 (Pin_4), J5.5 (Pin_5)
- net RX1P: now reaches J2.A2 (TX1+)
- net RX1P: now also C38.1
- net RX1N: now reaches J2.A3 (TX1-)
- net RX1N: now also C37.1
- net USB_DN: now reaches J2.A7 (D-)
- net TX1N: now reaches J2.B10 (RX1-)
- net TX1N: now also C35.1
- net TX1P: now reaches J2.B11 (RX1+)
- net TX1P: now also C36.1
- net GPIO14 renamed TYPEC_ORI
- net TYPEC_ORI: now also U9.2 (XSD)
- net TYPEC_RX2N renamed TX2N
- net TYPEC_RX2P renamed TX2P
- new net: C35.2, U9.19 (B0_P)
- new net: C16.2, U9.15 (C0_P)
- new net: C40.2, U9.12 (C1_N)
- new net: C39.2, U9.13 (C1_P)
- new net: C17.2, U9.14 (C0_N)
- new net: C38.2, U9.16 (B1_N)
- new net: C37.2, U9.17 (B1_P)
- new net: C36.2, U9.18 (B0_N)
- new net RX2N: C39.1, J2.B3 (TX2-)
- new net RX2P: C40.1, J2.B2 (TX2+)
- now unconnected: U5.A2 (VBUS)
- no-connect marks 29 -> 23
Other:
- note added: "SBU reverse is handled by PTN3460"
- note added: "Use PTN3460 reverse polarity"
- note added: "Vfb=0.6V"
- note added: "When using as display sink (UFP_D): Normal Fliped ML0 B2/3 A2/3 ML1 A11/10 B11/10 ML2 B11/10 A11/10 ML3 A2/3 B2/3"
- moved on the sheet: C1, C16, C17, C19, C26, C4, C6, J2, R2, R3, R4, R5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
